File: Hardware/airspeed_BIO/airspeed_BIO.kicad_pcb (KiCad board)
At the start: 2 copper layers, 50 x 35 mm, 91 parts, among them J1 USB_C_Receptacle_USB2.0_16P, J2 LOG_DEBUG, J3 BATT, J4 RF, Q1 2N7002, SW1 SW_SPDT, SW2 434123025826, SW3 434123025826, U1 MP2637GR-P, U2 LDL1117S33R, U3 2511020213301, U4 2513130810102, U5 2525020210002, U6 STM32F042G6Ux, U7 2607011111000, Y1 830108313809

Commit message: layoyt end
Parts:
- removed the C12 at (209.5, 112.4)
- removed the C16 at (169.8, 83.0)
- removed the C17 at (169.8, 85.5)
- removed the TP1 at (208.8, 115.4)
- C13: renamed from C14; moved to B.Cu
- C7, C8, C9, J4, U2, U7: moved to B.Cu
- moved TP2 92.0 mm to (138.0, 64.7)
- moved TP1 91.9 mm to (138.0, 68.0)
- moved J4 90.5 mm to (113.0, 64.0), turned to 180 degrees
- moved RLED1 87.8 mm to (120.4, 81.6), turned to 180 degrees
- moved C13 87.1 mm to (123.6, 80.4)
- moved C21 85.6 mm to (117.5, 65.7), turned to -90 degrees
- moved U2 85.3 mm to (121.9, 86.1), turned to 180 degrees
- moved C18 84.6 mm to (119.0, 65.7), turned to -90 degrees
- moved R20 83.1 mm to (120.4, 83.3)
- moved C27 79.4 mm to (121.3, 74.0), turned to -90 degrees
- moved C28 78.9 mm to (119.0, 74.0), turned to -90 degrees
- moved C19 76.6 mm to (105.5, 63.5), turned to 180 degrees
- moved U6 73.3 mm to (109.8, 80.0)
- moved C16 73.1 mm to (105.5, 65.0), turned to 180 degrees
- moved C17 69.8 mm to (112.0, 69.1)
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- renumbered C13 to C12, C15 to C14, C16 to C15, C17 to C16, C18 to C17, C19 to C18, C20 to C19, C21 to C20, C22 to C21, C23 to C22, C24 to C23, C25 to C24, C26 to C25, C27 to C26, C28 to C27, C29 to C28, TP2 to TP1, TP3 to TP2
Routing:
- net +3V3: track 0.00 -> 115.9 mm, vias 0 -> 9
- net GND: track 13.1 -> 90.6 mm, vias 0 -> 40
- net /MCU/I2C1.SCL: track 0.00 -> 43.9 mm, vias 0 -> 2
- net /MCU/I2C1.SDA: track 0.00 -> 43.3 mm, vias 0 -> 2
- net /MCU/SYS.SWCLK: track 0.00 -> 34.5 mm, vias 0 -> 2
- net /MCU/SYS.SWDIO: track 0.00 -> 34.3 mm, vias 0 -> 2
- net /MCU/NRST: track 0.00 -> 33.5 mm
- net /power/VCCpm: track 20.0 -> 49.3 mm, vias 1 -> 2
- net /MCU/USART1.RX: track 0.00 -> 26.5 mm
- net /connector/BATT: track 11.5 -> 37.3 mm, vias 0 -> 2
- net /MCU/USART2.CTS: track 0.00 -> 24.6 mm, vias 0 -> 1
- net Net-(U1-CSP): track 4.70 -> 29.0 mm, vias 0 -> 2
- net /MCU/USART1.TX: track 0.00 -> 21.6 mm
- net /MCU/USART2.RX: track 0.00 -> 18.7 mm, vias 0 -> 1
- net /MCU/USART2.TX: track 0.00 -> 18.4 mm, vias 0 -> 1
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- added copper zone on B.Cu, net +3V3
- added copper zone on B.Cu, net +5V
- added copper zone on B.Cu, net GND
- added copper zone on F.Cu, net GND
Other:
- board size 50 x 35 mm -> 54.5 x 39.5 mm
