File: Hardware/MCU.kicad_sch (KiCad schematic)
At the start: 10 parts, among them SW2 434123025826, U6 STM32F042G6Ux, Y1 830108313809

Commit message: fix pcb
Parts:
- C22, C23: MOUSER 80-CBR04C130F5GAC -> 80-CBR06C130F5GAC
- C24: MOUSER 80-C0402C105K4P -> 80-C0603C105K4P
- C26: MOUSER 80-C0402C104K4P -> 80-C0603C104J3REAULR
- R26: MOUSER 603-AC0402FR-070RL -> 603-AC0603FR-070RL
- R27: value 10k -> 10K; MOUSER 603-AC0402FR-0710KL -> (none)
Changed lines of the file:
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@@
 			)
 		)
-		(property "MOUSER" "80-CBR04C130F5GAC"
+		(property "MOUSER" "80-CBR06C130F5GAC"
 			(at 58.42 106.68 0)
 			(effects
@@
 			)
 		)
-		(property "MOUSER" "80-C0402C104K4P"
+		(property "MOUSER" "80-C0603C104J3REAULR"
 			(at 143.51 60.96 0)
 			(effects
@@
 			)
 		)
-		(property "MOUSER" "80-C0402C105K4P"
+		(property "MOUSER" "80-C0603C105K4P"
 			(at 81.28 68.58 0)
 			(effects
@@
 			)
 		)
-		(property "MOUSER" "80-CBR04C130F5GAC"
+		(property "MOUSER" "80-CBR06C130F5GAC"
 			(at 58.42 93.98 0)
 			(effects
@@
 			)
 		)
-		(property "MOUSER" "603-AC0402FR-070RL"
+		(property "MOUSER" "603-AC0603FR-070RL"
 			(at 74.93 106.68 0)
 			(effects
@@
 			)
 		)
-		(property "Value" "10k"
+		(property "Value" "10K"
 			(at 83.82 59.69 0)
 			(effects
@@
 			)
 		)
-		(property "MOUSER" "603-AC0402FR-0710KL"
+		(property "MOUSER" ""
 			(at 81.28 58.42 0)
 			(effects
