File: Hardware/airspeed_BIO.kicad_pcb (KiCad board)
At the start: 2 copper layers, 54.5 x 39.5 mm, 87 parts, among them J1 USB_C_Receptacle_USB2.0_16P, J2 LOG_DEBUG, J3 BATT, J4 RF, Q1 2N7002, SW1 SW_SPDT, SW2 434123025826, SW3 434123025826, U1 MP2637GR-P, U2 LDL1117S33R, U3 2511020213301, U4 2513130810102, U5 2525020210002, U6 STM32F042G6Ux, U7 2607011111000, Y1 830108313809

Commit message: fix pcb
Parts:
- added G***: LOGO, TTR:TTR_Logo, F.Cu at (108.7, 87.8)
Other:
- board text added: "V1.0"
- board text added: "design by Chen"
Changed lines of the file:
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@@
 			(outputformat 1)
 			(mirror no)
-			(drillshape 1)
+			(drillshape 0)
 			(scaleselection 1)
-			(outputdirectory "release/v1/")
+			(outputdirectory "release/v1/gerber/")
 		)
 	)
@@
 		)
 	)
+	(footprint "TTR:TTR_Logo"
+		(layer "F.Cu")
+		(at 108.65 87.8)
+		(property "Reference" "G***"
+			(at 0 0 0)
+			(layer "F.SilkS")
+			(hide yes)
+			(effects
+				(font
+					(size 1.5 1.5)
+					(thickness 0.3)
+				)
+			)
+		)
+		(property "Value" "LOGO"
+			(at 0.75 0 0)
+			(layer "F.SilkS")
+			(hide yes)
+			(effects
+				(font
+					(size 1.5 1.5)
+					(thickness 0.3)
+				)
+			)
+		)
+		(property "Datasheet" ""
+			(at 0 0 0)
+			(layer "F.Fab")
+			(hide yes)
+			(effects
+				(font
+					(size 1.27 1.27)
+					(thickness 0.15)
+				)
+			)
+		)
+		(property "Description" ""
+			(at 0 0 0)
+			(layer "F.Fab")
+			(hide yes)
+			(effects
+				(font
+					(size 1.27 1.27)
+					(thickness 0.15)
+				)
+			)
+		)
+		(attr board_only exclude_from_pos_files exclude_from_bom)
+		(fp_poly
+			(pts
+				(xy -1.510366 -2.931231) (xy -1.097887 -2.930547) (xy -0.717492 -2.92939) (xy -0.371889 -2.927785)
+				(xy -0.063785 -2.925755) (xy 0.204111 -2.923325) (xy 0.429092 -2.92052) (xy 0.608451 -2.917363)
+				(xy 0.739477 -2.91388) (xy 0.819465 -2.910096) (xy 0.845727 -2.906147) (xy 0.832167 -2.8757) (xy 0.79399 -2.803298)
+				(xy 0.734948 -2.69571) (xy 0.658792 -2.559704) (xy 0.569277 -2.40205) (xy 0.482388 -2.250709) (xy 0.119049 -1.620977)
+				(xy -0.158955 -1.603145) (xy -0.282046 -1.596995) (xy -0.445315 -1.591354) (xy -0.632557 -1.586647)
+				(xy -0.827568 -1.583302) (xy -0.959989 -1.582002) (xy -1.48302 -1.57869) (xy -2.778291 0.690677)
+				(xy -4.073563 2.960044) (xy -5.041181 2.960044) (xy -6.008798 2.960044) (xy -5.923793 2.812042)
+				(xy -5.897069 2.765663) (xy -5.844337 2.674286) (xy -5.7678 2.541725) (xy -5.669664 2.371798) (xy -5.552133 2.16832)
+				(xy -5.417412 1.935109) (xy -5.267704 1.675979) (xy -5.105216 1.394748) (xy -4.93215 1.095231) (xy -4.750712 0.781244)
+				(xy -4.600627 0.521532) (xy -3.362469 -1.620977) (xy -4.415752 -1.628363) (xy -4.653163 -1.630546)
+				(xy -4.871871 -1.633553) (xy -5.0657 -1.637225) (xy -5.228476 -1.6414) (xy -5.354025 -1.645917)
+				(xy -5.436172 -1.650616) (xy -5.468742 -1.655335) (xy -5.469034 -1.655812) (xy -5.45557 -1.68475)
+				(xy -5.417667 -1.7558) (xy -5.359058 -1.862235) (xy -5.283476 -1.997329) (xy -5.194656 -2.154354)
+				(xy -5.1096 -2.303427) (xy -4.750166 -2.93098) (xy -1.95222 -2.931417)
+			)
+			(stroke
+				(width 0)
+				(type solid)
+			)
+			(fill yes)
+			(layer "F.SilkS")
+		)
+		(fp_poly
+			(pts
+				(xy 3.59434 -2.931398) (xy 5.539512 -2.931303) (xy 5.685699 -2.863238) (xy 5.829804 -2.770698) (xy 5.9059 -2.683333)
+				(xy 5.968774 -2.548175) (xy 5.998169 -2.395225) (xy 5.991447 -2.246347) (xy 5.968303 -2.166443)
+				(xy 5.937118 -2.101936) (xy 5.881263 -1.99701) (xy 5.804284 -1.857697) (xy 5.709725 -1.690025) (xy 5.601133 -1.500026)
+				(xy 5.482051 -1.293729) (xy 5.356024 -1.077165) (xy 5.226598 -0.856365) (xy 5.097318 -0.637358)
+				(xy 4.971729 -0.426175) (xy 4.853376 -0.228845) (xy 4.745803 -0.051401) (xy 4.652556 0.10013) (xy 4.57718 0.219715)
+				(xy 4.523219 0.301325) (xy 4.49728 0.335853) (xy 4.335241 0.482936) (xy 4.138548 0.613827) (xy 3.928873 0.714761)
+				(xy 3.864187 0.737959) (xy 3.812225 0.753919) (xy 3.759473 0.766951) (xy 3.699484 0.777441) (xy 3.625811 0.785779)
+				(xy 3.532005 0.792353) (xy 3.411619 0.797551) (xy 3.258206 0.801762) (xy 3.065318 0.805373) (xy 2.826508 0.808772)
+				(xy 2.651969 0.810951) (xy 1.625025 0.823398) (xy 1.809523 0.920794) (xy 1.932429 0.994494) (xy 2.062287 1.085908)
+				(xy 2.14963 1.156882) (xy 2.202876 1.211117) (xy 2.285454 1.304001) (xy 2.392336 1.429479) (xy 2.518496 1.581496)
+				(xy 2.658906 1.753999) (xy 2.80854 1.940931) (xy 2.955782 2.127809) (xy 3.606324 2.960044) (xy 2.412388 2.960044)
+				(xy 1.218452 2.960044) (xy 1.013216 2.628801) (xy 0.814016 2.310026) (xy 0.638452 2.035371) (xy 0.482831 1.799644)
+				(xy 0.343454 1.597651) (xy 0.216627 1.4242) (xy 0.098653 1.274098) (xy -0.014163 1.142152) (xy -0.125517 1.02317)
+				(xy -0.140181 1.00828) (xy -0.439894 0.705684) (xy -1.219486 0.69818) (xy -1.999077 0.690677) (xy -1.711359 0.19068)
+				(xy -1.42364 -0.309318) (xy 0.511514 -0.309709) (xy 0.889601 -0.309836) (xy 1.215627 -0.310134)
+				(xy 1.493914 -0.31072) (xy 1.728782 -0.311711) (xy 1.924554 -0.313226) (xy 2.08555 -0.315382) (xy 2.216092 -0.318297)
+				(xy 2.320501 -0.32209) (xy 2.403098 -0.326878) (xy 2.468204 -0.332779) (xy 2.52014 -0.33991) (xy 2.563228 -0.348391)
+				(xy 2.60179 -0.358338) (xy 2.632734 -0.367569) (xy 2.760311 -0.417443) (xy 2.876313 -0.487679) (xy 2.98699 -0.584702)
+				(xy 3.098596 -0.714939) (xy 3.217382 -0.884818) (xy 3.349598 -1.100766) (xy 3.35507 -1.110135) (xy 3.44053 -1.261349)
+				(xy 3.507978 -1.390134) (xy 3.553743 -1.488956) (xy 3.574157 -1.55028) (xy 3.57468 -1.561189) (xy 3.566149 -1.620977)
+				(xy 2.230906 -1.611309) (xy 1.884117 -1.609306) (xy 1.592284 -1.608736) (xy 1.353998 -1.60962) (xy 1.167852 -1.61198)
+				(xy 1.032438 -1.615836) (xy 0.946346 -1.62121) (xy 0.908171 -1.628123) (xy 0.905934 -1.631158) (xy 0.922293 -1.662675)
+				(xy 0.963054 -1.73618) (xy 1.024364 -1.844871) (xy 1.10237 -1.981948) (xy 1.193216 -2.140607) (xy 1.282686 -2.296084)
+				(xy 1.649168 -2.931494)
+			)
+			(stroke
+				(width 0)
+				(type solid)
+			)
+			(fill yes)
+			(layer "F.SilkS")
+		)
+		(embedded_fonts no)
+	)
 	(footprint "Resistor_SMD:R_0603_1608Metric"
 		(layer "F.Cu")
@@
 		)
 	)
+	(gr_rect
+		(start 114.7 89)
+		(end 118.4 90.7)
+		(stroke
+			(width 0.3)
+			(type solid)
+		)
+		(fill no)
+		(layer "F.SilkS")
+	)
 	(gr_arc
 		(start 98 100)
@@
 		(layer "Edge.Cuts")
 	)
+	(gr_text "V1.0"
+		(at 114.9 90.5 0)
+		(layer "F.SilkS")
+		(effects
+			(font
+				(size 1 1)
+				(thickness 0.2)
+				(bold yes)
+			)
+			(justify left bottom)
+		)
+	)
+	(gr_text "design by Chen"
+		(at 113.7 98 0)
+		(layer "B.SilkS")
+		(effects
+			(font
+				(size 1 1)
+				(thickness 0.2)
+				(bold yes)
+			)
+			(justify left bottom mirror)
+		)
+	)
 	(segment
