File: Hardware/power.kicad_sch (KiCad schematic)
At the start: 42 parts, among them Q1 2N7002, U1 MP2637GR-P, U2 LDL1117S33R

Commit message: fix pcb
Parts:
- C6: value 100nF -> 0.1u; MOUSER (none) -> 80-C0603C104J3REAULR
- L1: MOUSER (none) -> https://www.mouser.tw/ProductDetail/Vishay-Dale/IHLP1210BZE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; Mouser https://www.mouser.tw/ProductDetail/Vishay-Dale/IHLP1210BZE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 -> (none)
- R15: MOUSER (none) -> https://www.mouser.tw/ProductDetail/YAGEO/PE1206FRE470R02L?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; Mouser https://www.mouser.tw/ProductDetail/YAGEO/PE1206FRE470R02L?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 -> (none)
- R9: MOUSER (none) -> 603-AC0603FR-070RL
- U1: MOUSER (none) -> https://www.mouser.tw/ProductDetail/Monolithic-Power-System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; Mouser https://www.mouser.tw/ProductDetail/Monolithic-Power-System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 -> (none)
Changed lines of the file:
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@@
 			)
 		)
-		(property "Mouser" "https://www.mouser.tw/ProductDetail/Vishay-Dale/IHLP1210BZEZ2R2M5A?qs=iLKYxzqNS75fATvQbHxN2g%3D%3D"
+		(property "Mouser" ""
+			(at 157.48 88.9 90)
+			(effects
+				(font
+					(size 1.27 1.27)
+				)
+				(hide yes)
+			)
+		)
+		(property "MOUSER" "https://www.mouser.tw/ProductDetail/Vishay-Dale/IHLP1210BZEZ2R2M5A?qs=iLKYxzqNS75fATvQbHxN2g%3D%3D"
 			(at 157.48 88.9 90)
 			(effects
@@
 			)
 		)
-		(property "Mouser" "https://www.mouser.tw/ProductDetail/Monolithic-Power-Systems-MPS/MP2637GR-P?qs=493kPxzlxfIVMFQDxi%252BdaQ%3D%3D"
+		(property "Mouser" ""
 			(at 129.032 148.844 0)
 			(effects
@@
 			)
 		)
+		(property "MOUSER" "https://www.mouser.tw/ProductDetail/Monolithic-Power-Systems-MPS/MP2637GR-P?qs=493kPxzlxfIVMFQDxi%252BdaQ%3D%3D"
+			(at 128.27 107.95 0)
+			(effects
+				(font
+					(size 1.27 1.27)
+				)
+				(hide yes)
+			)
+		)
 		(pin "20"
 		)
@@
 			)
 		)
-		(property "Mouser" "https://www.mouser.tw/ProductDetail/YAGEO/PE1206FRE470R02L?qs=eP2BKZSCXI6QA3qQIx2m4A%3D%3D"
+		(property "Mouser" ""
+			(at 171.45 88.9 90)
+			(effects
+				(font
+					(size 1.27 1.27)
+				)
+				(hide yes)
+			)
+		)
+		(property "MOUSER" "https://www.mouser.tw/ProductDetail/YAGEO/PE1206FRE470R02L?qs=eP2BKZSCXI6QA3qQIx2m4A%3D%3D"
 			(at 171.45 88.9 90)
 			(effects
@@
 			)
 		)
-		(property "Value" "100nF"
+		(property "Value" "0.1u"
 			(at 157.48 133.3562 0)
 			(effects
@@
 			)
 		)
+		(property "MOUSER" "80-C0603C104J3REAULR"
+			(at 154.94 132.08 0)
+			(effects
+				(font
+					(size 1.27 1.27)
+				)
+				(hide yes)
+			)
+		)
+		(property "WE" ""
+			(at 154.94 132.08 0)
+			(effects
+				(font
+					(size 1.27 1.27)
+				)
+				(hide yes)
+			)
+		)
 		(pin "1"
 		)
@@
 			(at 128.27 73.66 0)
 			(effects
+				(font
+					(size 1.27 1.27)
+				)
+				(hide yes)
+			)
+		)
+		(property "MOUSER" "603-AC0603FR-070RL"
+			(at 128.27 73.66 0)
+			(effects
